File: PCB Design/AD3551R_DAC/AD3551R_DAC.kicad_sch (KiCad schematic)
At the start: 22 parts, among them J101 RJ45_LED_Shielded, J102 RJ45_LED_Shielded, J103 Screw_Terminal_01x02, J104 USB_C_Receptacle_USB2.0_14P, J105 Conn_Coaxial, SW101 SW_SPDT, SW102 SW_SPDT

Commit message: Placement Done
Placement Done
Parts:
- removed R101, R102, R103, R104: 220, Resistor_SMD:R_0603_1608Metric_Pad0.98x0.95mm_HandSolder, symbol Device:R_Small
Connections:
- net GND: no longer J101.11, J101.9, J102.11, J102.9
- no-connect marks 4 -> 12

Commit message: Layout changes + Aesthetic
Layout changes + Aesthetic
Parts:
- J101, J102: footprint Connector_RJ:RJ45_Abracon_ARJP11A-MA_Horizontal -> Connector_RJ:RJ45_Amphenol_RJHSE538X
Connections:
- net GND: now also J101.5, J102.5; no longer J101.4, J102.4
- net SPI_Communication/3.3VSDIO2: now also J101.4; no longer J101.5
- net SPI_Communication/3.3V_SDI: now also J102.4; no longer J102.5
Changed lines of the file:
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@@
 	(wire
 		(pts
-			(xy 55.88 44.45) (xy 81.28 44.45)
+			(xy 191.77 52.07) (xy 191.77 49.53)
 		)
 		(stroke
-			(width 0.254)
+			(width 0.508)
 			(type default)
-			(color 0 0 255 1)
+			(color 0 0 194 1)
 		)
 	)
 	(wire
 		(pts
-			(xy 191.77 52.07) (xy 191.77 49.53)
+			(xy 78.74 57.15) (xy 101.6 57.15)
 		)
 		(stroke
-			(width 0.508)
+			(width 0.254)
 			(type default)
-			(color 0 0 194 1)
+			(color 0 0 255 1)
 		)
 	)
 	(wire
 		(pts
-			(xy 81.28 57.15) (xy 101.6 57.15)
+			(xy 78.74 46.99) (xy 55.88 46.99)
 		)
 		(stroke
@@
 	(wire
 		(pts
+			(xy 55.88 80.01) (xy 73.66 80.01)
+		)
+		(stroke
+			(width 0)
+			(type default)
+		)
+	)
+	(wire
+		(pts
 			(xy 133.35 59.69) (xy 149.86 59.69)
 		)
@@
 	(wire
 		(pts
-			(xy 83.82 54.61) (xy 83.82 41.91)
+			(xy 85.09 54.61) (xy 85.09 41.91)
 		)
 		(stroke
@@
 	(wire
 		(pts
+			(xy 78.74 57.15) (xy 78.74 46.99)
+		)
+		(stroke
+			(width 0.254)
+			(type default)
+			(color 0 0 255 1)
+		)
+	)
+	(wire
+		(pts
 			(xy 191.77 49.53) (xy 191.77 43.18)
 		)
@@
 	(wire
 		(pts
-			(xy 55.88 46.99) (xy 78.74 46.99)
-		)
-		(stroke
-			(width 0)
-			(type default)
-		)
-	)
-	(wire
-		(pts
 			(xy 208.28 64.77) (xy 208.28 66.04)
 		)
@@
 	(wire
 		(pts
-			(xy 55.88 41.91) (xy 83.82 41.91)
+			(xy 55.88 41.91) (xy 85.09 41.91)
 		)
 		(stroke
@@
 	(wire
 		(pts
-			(xy 101.6 67.31) (xy 92.71 67.31)
+			(xy 101.6 67.31) (xy 93.98 67.31)
 		)
 		(stroke
@@
 	(wire
 		(pts
-			(xy 81.28 110.49) (xy 83.82 110.49)
+			(xy 93.98 67.31) (xy 93.98 82.55)
 		)
 		(stroke
-			(width 0.508)
+			(width 0.254)
 			(type default)
-			(color 255 0 255 1)
+			(color 0 0 255 1)
 		)
 	)
 	(wire
 		(pts
-			(xy 41.91 157.48) (xy 41.91 156.21)
+			(xy 55.88 44.45) (xy 81.28 44.45)
 		)
 		(stroke
@@
 	(wire
 		(pts
-			(xy 92.71 80.01) (xy 55.88 80.01)
+			(xy 81.28 110.49) (xy 83.82 110.49)
 		)
 		(stroke
-			(width 0.254)
+			(width 0.508)
+			(type default)
+			(color 255 0 255 1)
+		)
+	)
+	(wire
+		(pts
+			(xy 41.91 157.48) (xy 41.91 156.21)
+		)
+		(stroke
+			(width 0)
 			(type default)
-			(color 0 0 255 1)
 		)
 	)
@@
 	(wire
 		(pts
-			(xy 101.6 54.61) (xy 83.82 54.61)
+			(xy 93.98 82.55) (xy 55.88 82.55)
 		)
 		(stroke
@@
 	(wire
 		(pts
-			(xy 49.53 157.48) (xy 41.91 157.48)
+			(xy 101.6 54.61) (xy 85.09 54.61)
 		)
 		(stroke
-			(width 0)
+			(width 0.254)
 			(type default)
+			(color 0 0 255 1)
 		)
 	)
 	(wire
 		(pts
-			(xy 181.61 64.77) (xy 191.77 64.77)
+			(xy 49.53 157.48) (xy 41.91 157.48)
 		)
 		(stroke
@@
 	(wire
 		(pts
-			(xy 59.69 176.53) (xy 48.26 176.53)
+			(xy 181.61 64.77) (xy 191.77 64.77)
 		)
 		(stroke
-			(width 0.508)
+			(width 0)
 			(type default)
-			(color 255 255 0 1)
 		)
 	)
 	(wire
 		(pts
-			(xy 92.71 67.31) (xy 92.71 80.01)
+			(xy 59.69 176.53) (xy 48.26 176.53)
 		)
 		(stroke
-			(width 0.254)
+			(width 0.508)
 			(type default)
-			(color 0 0 255 1)
+			(color 255 255 0 1)
 		)
 	)
@@
 	(wire
 		(pts
-			(xy 55.88 82.55) (xy 72.39 82.55)
-		)
-		(stroke
-			(width 0)
-			(type default)
-		)
-	)
-	(wire
-		(pts
 			(xy 49.53 158.75) (xy 49.53 157.48)
 		)
@@
 	(wire
 		(pts
-			(xy 81.28 57.15) (xy 81.28 44.45)
-		)
-		(stroke
-			(width 0.254)
-			(type default)
-			(color 0 0 255 1)
-		)
-	)
-	(wire
-		(pts
 			(xy 101.6 62.23) (xy 87.63 62.23)
 		)
@@
 			)
 		)
-		(property "Footprint" "Connector_RJ:RJ45_Abracon_ARJP11A-MA_Horizontal"
+		(property "Footprint" "Connector_RJ:RJ45_Amphenol_RJHSE538X"
 			(at 45.72 46.355 90)
 			(hide yes)
@@
 	(symbol
 		(lib_id "power:GND")
-		(at 78.74 46.99 0)
+		(at 81.28 44.45 0)
 		(unit 1)
 		(body_style 1)
@@
 		(fields_autoplaced yes)
 		(property "Reference" "#PWR0106"
-			(at 78.74 53.34 0)
+			(at 81.28 50.8 0)
 			(hide yes)
 			(show_name no)
@@
 		)
 		(property "Value" "GND"
-			(at 78.74 52.07 0)
+			(at 81.28 49.53 0)
 			(hide yes)
 			(show_name no)
@@
 		)
 		(property "Footprint" ""
-			(at 78.74 46.99 0)
+			(at 81.28 44.45 0)
 			(hide yes)
 			(show_name no)
@@
 		)
 		(property "Datasheet" ""
-			(at 78.74 46.99 0)
+			(at 81.28 44.45 0)
 			(hide yes)
 			(show_name no)
@@
 		)
 		(property "Description" "Power symbol creates a global label with name \"GND\" , ground"
-			(at 78.74 46.99 0)
+			(at 81.28 44.45 0)
 			(hide yes)
 			(show_name no)
@@
 	(symbol
 		(lib_id "power:GND")
-		(at 72.39 82.55 0)
+		(at 73.66 80.01 0)
 		(unit 1)
 		(body_style 1)
@@
 		(fields_autoplaced yes)
 		(property "Reference" "#PWR0109"
-			(at 72.39 88.9 0)
+			(at 73.66 86.36 0)
 			(hide yes)
 			(show_name no)
@@
 		)
 		(property "Value" "GND"
-			(at 72.39 87.63 0)
+			(at 73.66 85.09 0)
 			(hide yes)
 			(show_name no)
@@
 		)
 		(property "Footprint" ""
-			(at 72.39 82.55 0)
+			(at 73.66 80.01 0)
 			(hide yes)
 			(show_name no)
@@
 		)
 		(property "Datasheet" ""
-			(at 72.39 82.55 0)
+			(at 73.66 80.01 0)
 			(hide yes)
 			(show_name no)
@@
 		)
 		(property "Description" "Power symbol creates a global label with name \"GND\" , ground"
-			(at 72.39 82.55 0)
+			(at 73.66 80.01 0)
 			(hide yes)
 			(show_name no)
@@
 			)
 		)
-		(property "Footprint" "Connector_RJ:RJ45_Abracon_ARJP11A-MA_Horizontal"
+		(property "Footprint" "Connector_RJ:RJ45_Amphenol_RJHSE538X"
 			(at 45.72 81.915 90)
 			(hide yes)

Commit message: Routing Done
Routing Done
Parts:
- removed TP101: TestPoint, TestPoint:TestPoint_Plated_Hole_D2.0mm, symbol Connector:TestPoint
Connections:
- no-connect marks 12 -> 13
Changed lines of the file:
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@@
+	)
+	(no_connect
+		(at 208.28 64.77)
 	)
 	(no_connect
@@
 					(unit 1)
 				)
-			)
-		)
-	)
-	(symbol
-		(lib_id "Connector:TestPoint")
-		(at 208.28 64.77 0)
-		(unit 1)
-		(body_style 1)
-		(exclude_from_sim no)
-		(in_bom yes)
-		(on_board yes)
-		(in_pos_files yes)
-		(dnp no)
-		(property "Reference" "TP101"
-			(at 209.55 64.77 0)
-			(show_name no)
-			(do_not_autoplace no)
-			(effects
-				(font
-					(size 1.27 1.27)
-				)
-				(justify left)
-			)
-		)
-		(property "Value" "TestPoint"
-			(at 210.82 62.738 0)
-			(hide yes)
-			(show_name no)
-			(do_not_autoplace no)
-			(effects
-				(font
-					(size 1.27 1.27)
-				)
-				(justify left)
-			)
-		)
-		(property "Footprint" "TestPoint:TestPoint_Plated_Hole_D2.0mm"
-			(at 213.36 64.77 0)
-			(hide yes)
-			(show_name no)
-			(do_not_autoplace no)
-			(effects
-				(font
-					(size 1.27 1.27)
-				)
-			)
-		)
-		(property "Datasheet" ""
-			(at 213.36 64.77 0)
-			(hide yes)
-			(show_name no)
-			(do_not_autoplace no)
-			(effects
-				(font
-					(size 1.27 1.27)
-				)
-			)
-		)
-		(property "Description" "test point"
-			(at 208.28 64.77 0)
-			(hide yes)
-			(show_name no)
-			(do_not_autoplace no)
-			(effects
-				(font
-					(size 1.27 1.27)
-				)
-			)
-		)
-		(pin "1"
-		)
-		(instances
-			(project "AD3551R_DAC"
-				(path "/3d4144e0-3656-4efa-94fd-8cd1f0e2cd3f"
-					(reference "TP101")
-					(unit 1)
-				)
