File: PCB Design/AD3551R_DAC/AD3551R_DAC.kicad_pcb (KiCad board)
At the start: 4 copper layers, 100 x 100 mm, 89 parts, among them J101 RJ45_LED_Shielded, J102 RJ45_LED_Shielded, J103 Screw_Terminal_01x02, J104 USB_C_Receptacle_USB2.0_14P, J105 Conn_Coaxial, SW101 SW_SPDT, SW102 SW_SPDT, SW201 SW_SPDT, SW202 SW_SPDT, SW301 SW_SPDT, SW302 SW_DP3T, SW303 SW_SPDT, SW401 SW_SPDT, SW402 SW_SPDT, SW403 SW_SPDT, SW404 SW_SPDT, U201 TXB0101DBV, U202 TXB0101DBV, U203 TXB0101DBV, U204 TXB0101DBV, U205 TXB0101DBV, U206 TXB0101DBV, U301 AD3551RBCPZ16, U303 AD8065ARTZ-R2, U402 AP63203WU, U403 AP63205WU

Commit message: Placement Done
Placement Done
Parts:
- removed R101, R102, R103, R104: 220, Resistor_SMD:R_0603_1608Metric_Pad0.98x0.95mm_HandSolder
- added U401: TLV75718PDYDR, Parts_fab:TLV_1V8, F.Cu at (136.9, 132.8)
- moved R301 218.9 mm to (58.0, 75.1), turned to -90 degrees
- moved R202 194.3 mm to (58.1, 129.8), turned to 90 degrees
- moved R107 190.3 mm to (76.0, 136.3)
- moved R105 189.6 mm to (78.6, 138.7), turned to -90 degrees
- moved R201 187.9 mm to (65.0, 140.1), turned to 90 degrees
- moved C101 187.1 mm to (76.1, 140.0), turned to 180 degrees
- moved R106 186.1 mm to (81.6, 138.7), turned to -90 degrees
- moved D101 180.7 mm to (76.0, 138.2)
- moved U403 121.9 mm to (107.0, 137.0), turned to 90 degrees
- moved C409 119.9 mm to (102.5, 136.5), turned to -90 degrees
- moved C411 118.2 mm to (104.8, 121.1)
- moved C410 117.7 mm to (104.8, 123.3)
- moved C407 112.5 mm to (110.3, 137.8), turned to 90 degrees
- moved L402 110.6 mm to (104.8, 128.0), turned to 180 degrees
- moved R407 109.8 mm to (98.1, 136.5), turned to 90 degrees
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Connections:
- J101 pad 10: Net-(J101-Pad10) -> unconnected-(J101-Pad10)
- J101 pad 11: GND -> unconnected-(J101-Pad11)
- J101 pad 12: Net-(J101-Pad12) -> unconnected-(J101-Pad12)
- J101 pad 9: GND -> unconnected-(J101-Pad9)
- J102 pad 10: Net-(J102-Pad10) -> unconnected-(J102-Pad10)
- J102 pad 11: GND -> unconnected-(J102-Pad11)
- J102 pad 12: Net-(J102-Pad12) -> unconnected-(J102-Pad12)
- J102 pad 9: GND -> unconnected-(J102-Pad9)
Routing:
- net GND: vias 882 -> 810
Other:
- board text added: "+1.8V LDO"
- board text added: "+3.3V Switching"
- board text added: "+5V Switching"
- board text added: "Testing Procedure"

Commit message: more layout
more layout
Routing:
- net Net-(SW202-A): track 0.00 -> 5.10 mm
- net /Power/SW: track 0.00 -> 3.04 mm
- net Net-(U403-BST): track 0.00 -> 3.01 mm
- net /Power/BST: track 0.00 -> 2.93 mm
- net Net-(U403-SW): track 0.00 -> 2.82 mm
- net GND: vias 810 -> 1531
- added copper zone on F.Cu, net /Power/FB
- added copper zone on F.Cu, net Net-(SW403-B)
- added copper zone on F.Cu, net Net-(U403-FB)
- added copper zone on F.Cu, net Net-(U403-SW)
- added copper zone on F.Cu, net VSWITCH

Commit message: layout changes
layout changes soldermask sectioning done
Parts:
- moved C404 2.59 mm to (126.0, 135.5), turned to 180 degrees
- moved C401 1.04 mm to (133.0, 132.0), turned to 180 degrees
Routing:
- net Net-(SW401-B): track 0.00 -> 8.86 mm
- net Net-(SW201-A): track 0.00 -> 5.10 mm
- net Net-(SW402-C): track 0.00 -> 3.81 mm
- net Net-(SW403-C): track 0.00 -> 3.63 mm
- net Net-(SW401-C): track 0.00 -> 2.93 mm
- net Net-(D403-A): track 0.00 -> 2.01 mm
- net Net-(D402-A): track 0.00 -> 1.71 mm
- net /Power/SW: track 3.04 -> 4.07 mm
- net /Power/BST: track 2.93 -> 2.26 mm
- net /DAC_Main/1V8SCLK: track 22.6 -> 22.1 mm
- net GND: vias 1531 -> 1960
- added copper zone on F.Cu, net +3.3V
- added copper zone on F.Cu, net /Power/SW
- added copper zone on F.Cu, net Net-(SW401-B)
Other:
- board text added: "DAC/VTUNE OUT"
- board text added: "Flatrim Dreshaj 2026"
- board text added: "High Speed DAC"

Commit message: Layout changes + Aesthetic
Layout changes + Aesthetic
Parts:
- removed SW302: SW_DP3T, Parts_fab:3_way_switch_CUS-13TB_NDC
- J101, J102: footprint Connector_RJ:RJ45_Abracon_ARJP11A-MA_Horizontal -> Connector_RJ:RJ45_Amphenol_RJHSE538X
- moved J101 15.0 mm to (59.1, 95.6), turned to 90 degrees
- moved J102 13.4 mm to (59.1, 115.4), turned to 90 degrees
- moved C312 6.45 mm to (109.2, 93.6), turned to -90 degrees
- moved C310 3.63 mm to (107.2, 93.6), turned to -90 degrees
- moved C311 1.21 mm to (105.5, 93.6), turned to -90 degrees
Connections:
- J101 pad 4: GND -> /SPI_Communication/3.3VSDIO2
- J101 pad 5: /SPI_Communication/3.3VSDIO2 -> GND
- J102 pad 4: GND -> /SPI_Communication/3.3V_SDI
- J102 pad 5: /SPI_Communication/3.3V_SDI -> GND
Routing:
- net Net-(SW301-C): track 6.04 -> 49.0 mm
- net /SPI_Communication/3.3VSDIO3: track 0.00 -> 31.0 mm, vias 0 -> 1
- net /SPI_Communication/3.3VSDIO2: track 0.00 -> 30.1 mm, vias 0 -> 1
- net /SPI_Communication/3.3V_SCLK: track 0.00 -> 25.7 mm, vias 0 -> 1
- net /SPI_Communication/3.3V_SDI: track 0.00 -> 24.1 mm, vias 0 -> 1
- net /SPI_Communication/3.3VSDO: track 0.00 -> 14.1 mm
- net /SPI_Communication/VCCA_SPI: track 0.00 -> 14.0 mm
- net /SPI_Communication/3.3VCS1: track 0.00 -> 14.0 mm
- net GND: track 26.1 -> 24.0 mm, vias 1960 -> 1842

Commit message: power layout
power layout
Routing:
- net Net-(SW403-B): track 0.00 -> 55.7 mm, vias 0 -> 1
- net /Power/FB: track 0.00 -> 37.1 mm, vias 0 -> 5
- net +3.3V: track 0.00 -> 24.3 mm, vias 0 -> 3
- net GND: vias 1842 -> 1714

Commit message: Routing Done
Routing Done
Parts:
- removed TP101: TestPoint, TestPoint:TestPoint_Plated_Hole_D2.0mm
- moved SW102 10.5 mm to (131.0, 147.0), turned to 180 degrees
- moved SW101 9.00 mm to (122.0, 147.0), turned to 0 degrees
- moved TP102 2.85 mm to (101.5, 109.0)
- moved R105 0.69 mm to (78.5, 138.0)
- moved R106 0.68 mm to (81.6, 138.0)
- moved SW404 0.25 mm to (105.0, 147.0)
Connections:
- SW102 pad 1: Net-(SW102-A) -> unconnected-(SW102-A-Pad1)
- U301 pad 23: Net-(U301-RFB4__0) -> unconnected-(U301-RFB4__0-Pad23)
- U301 pad 24: Net-(U301-RFB2__0) -> /DAC_Main/DAC_OUT
- U301 pad 25: Net-(U301-RFB1__0) -> unconnected-(U301-RFB1__0-Pad25)
Routing:
- net +1V8: track 16.3 -> 239.7 mm, vias 0 -> 11
- net /SPI_Communication/OE: track 0.00 -> 94.5 mm, vias 0 -> 8
- net Net-(SW101-C): track 0.00 -> 81.7 mm
- net VSWITCH: track 0.00 -> 72.0 mm, vias 0 -> 2
- net /DAC_Main/1V8CS1: track 23.6 -> 92.7 mm, vias 0 -> 2
- net /DAC_Main/RESET: track 0.00 -> 63.9 mm, vias 0 -> 1
- net /DAC_Main/LDAC: track 0.00 -> 56.3 mm, vias 0 -> 1
- net Net-(SW303-B): track 0.00 -> 55.9 mm, vias 0 -> 1
- net /SPI_Communication/VCCA_SPI: track 14.0 -> 67.4 mm, vias 0 -> 7
- net +5V: track 5.54 -> 52.5 mm, vias 0 -> 2
- net VBUS: track 0.00 -> 43.1 mm, vias 0 -> 1
- net VSCREW: track 0.00 -> 12.0 mm
- net /DAC_Main/DAC_OUT: track 39.9 -> 48.6 mm
- net Net-(SW303-A): track 0.00 -> 4.99 mm
- net Net-(J104-CC1): track 0.00 -> 3.08 mm
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- added copper zone on F.Cu, net VBUS
- added copper zone on F.Cu, net VSCREW

Commit message: more changes
more changes
Connections:
- J104 pad : (no net) -> VBUS
- J104 pad A1_B12: (no net) -> VBUS
- J104 pad B1_A12: (no net) -> VBUS
- J104 pad B4_A9: (no net) -> VBUS
Routing:
- net /Power/FB: track 37.1 -> 43.7 mm, vias 3 -> 6
- net VSWITCH: track 72.0 -> 75.8 mm, vias 2 -> 3
- net +1V8: track 239.7 -> 237.6 mm
- net VBUS: track 43.1 -> 43.9 mm
- net GND: vias 1677 -> 1701
- net +3.3V: vias 3 -> 1
- added copper zone on In2.Cu, net /Power/FB
Other:
- board text added: "Ethernet SPI IN"
- board text added: "USBC IN"

Commit message: small changes
small changes
Connections:
- J104 pad : VBUS -> (no net)
- J104 pad A1_B12: VBUS -> (no net)
- J104 pad B1_A12: VBUS -> (no net)
- J104 pad B4_A9: VBUS -> (no net)
- U301 pad 23: unconnected-(U301-RFB4__0-Pad23) -> /DAC_Main/DAC_OUT
- U301 pad 24: /DAC_Main/DAC_OUT -> unconnected-(U301-RFB2__0-Pad24)
Routing:
- net VBUS: track 43.9 -> 23.7 mm
- net VSCREW: track 12.0 -> 15.8 mm
- net Net-(SW403-B): track 55.8 -> 55.0 mm
- net VSWITCH: vias 3 -> 2
- net GND: vias 1701 -> 1709
