File: PCB Design/AD3551R_DAC/AD3551R_DAC.kicad_pcb (KiCad board)
At the start: 4 copper layers, 100 x 100 mm, 84 parts, among them J101 RJ45_LED_Shielded, J102 RJ45_LED_Shielded, J103 Screw_Terminal_01x02, J104 USB_C_Receptacle_USB2.0_14P, J105 Conn_Coaxial, SW101 SW_SPDT, SW102 SW_SPDT, SW201 SW_SPDT, SW202 SW_SPDT, SW301 SW_SPDT, SW303 SW_SPDT, SW401 SW_SPDT, SW402 SW_SPDT, SW403 SW_SPDT, SW404 SW_SPDT, U201 TXB0101DBV, U202 TXB0101DBV, U203 TXB0101DBV, U204 TXB0101DBV, U205 TXB0101DBV, U206 TXB0101DBV, U301 AD3551RBCPZ16, U303 AD8065ARTZ-R2, U401 TLV75718PDYDR, U402 AP63203WU, U403 AP63205WU

Commit message: layout
layout
Connections:
- J104 pad SH1: (no net) -> GND
- J104 pad SH2: (no net) -> GND
- J104 pad SH3: (no net) -> GND
- J104 pad SH4: (no net) -> GND
Routing:
- net VBUS: track 23.7 -> 49.1 mm
- net +1V8: track 237.6 -> 219.8 mm
- net GND: track 26.6 -> 26.8 mm, vias 1709 -> 1704
- removed copper zone on F.Cu, net VBUS

Commit message: final touches
final touches
Routing:
- net GND: vias 1704 -> 1690
Other:
- board text added: "+5-23V"
- board text added: "GND | LDAC"
- board text added: "OFF AMP ON"
- board text added: "OFF LSHIFT ON"
- board text added: "ON +3V3 OFF"
- board text added: "ON +5V OFF"
- board text added: "RESET | FLOAT"
- board text added: "VSCREW | USB"
- board text added: "{dblquote}One must imagine Sisyphus happy.{dblquote} - Camus"
