File: PCB Design/AD3551R_DAC/DAC_Main.kicad_sch (KiCad schematic)
At the start: 17 parts, among them SW301 SW_SPDT, SW302 SW_SPDT, U301 AD3551RBCPZ16, U302 AD8065ARTZ-R2

Commit message: added comments for future changes on unnecesary components
added comments for future changes on unnecesary components
Other:
- note added: "unnecesary"
- note added: "unnecesary, tie to gnd"
