File: PCB Design/AD3551R_DAC/ad3551rb.kicad_sch (KiCad schematic)
At the start: 17 parts, among them J101 RJ45_LED_Shielded, J102 RJ45_LED_Shielded, J103 Conn_Coaxial, J104 USB_C_Receptacle_USB2.0_14P, J105 Screw_Terminal_01x02, SW101 SW_SPDT, SW102 SW_SPDT

Commit message: added comments for future changes on unnecesary components
added comments for future changes on unnecesary components
Other:
- note added: "SDIO 2 and 3 are Unnecesary remove and pull down"
- note added: "Unnecesary Tie to VLOGIC"
- note added: "unnecesary, tie to gnd"
Changed lines of the file:
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@@
 		)
 	)
+	(text "SDIO 2 and 3 are Unnecesary remove and pull down"
+		(exclude_from_sim no)
+		(at 51.562 65.786 0)
+		(effects
+			(font
+				(size 1.27 1.27)
+			)
+		)
+	)
+	(text "Unnecesary\nTie to VLOGIC"
+		(exclude_from_sim no)
+		(at 197.612 75.946 0)
+		(effects
+			(font
+				(size 1.27 1.27)
+			)
+		)
+	)
 	(text "Unnecesary -- remove next rev"
 		(exclude_from_sim no)
@@
 		)
 	)
+	(text "unnecesary, tie to gnd\n"
+		(exclude_from_sim no)
+		(at 157.48 98.552 0)
+		(effects
+			(font
+				(size 2.54 2.54)
+			)
+		)
+	)
 	(text "LEVEL SHIFTERS"
 		(exclude_from_sim no)
@@
 		)
 		(fill
-			(color 0 0 194 0.5019607843)
+			(color 0 255 255 1)
 		)
 		(property "Sheetname" "SPI_Communication [3]"
