File: TX_ADAR/powerdelivery.kicad_sch (KiCad schematic)
At the start: 19 parts, among them U1 LT1761-1.8, U3 LT1761-2.5

Commit message: Cleaning up schematic
Added Cal Line
Connected RFOuts to connectors
Worked on State Machine connections
Finished connecting SDP Connector (need to double check)
Parts:
- removed C1, C14, C4: 1uF, symbol Device:C_Small_US
- removed C10, C12, C15, C8: 10nF, symbol Device:C_Small_US
- removed C11, C13, C16, C9: 100pF, symbol Device:C_Small_US
- removed C2, C5: 0.01uF, symbol Device:C_Small_US
- removed C3, C6: 10uF, symbol Device:C_Small_US
- added C10, C15: 0.01uF, symbol Device:C
- added C11, C43: 10uF, symbol Device:C
- added C14, C7: 1uF, symbol Device:C
Connections:
- net 1V8: now also C10.1, C11.1
- net 5V: now also C14.1, C7.1
- net GND: now also C11.2, C14.2, C43.2, C7.2
- net at U3.4 (BYP): now also C15.2
- net at U1.4 (BYP): now also C10.2
- net VPOS renamed 2V5
- net 2V5: now also C15.1, C43.1
Other:
- note removed: "Decoupling Caps for 2V5 (As close as possible to pins)"

Commit message: Fixing problems pointed out
Parts:
- removed C10, C15: 0.01uF, symbol Device:C
- removed C11, C43: 10uF, symbol Device:C
- removed C14, C7: 1uF, symbol Device:C
- removed U1: LT1761-1.8, Package_TO_SOT_SMD:TSOT-23-5, symbol Regulator_Linear:LT1761-1.8
- removed U3: LT1761-2.5, Package_TO_SOT_SMD:TSOT-23-5, symbol Regulator_Linear:LT1761-2.5
- added C1, C2, C3, C4: 10uF, Package_SO:SOIC-8_3.9x4.9mm_P1.27mm, symbol Device:C
- added IC1: REG1117A-1.8, Package_DFN_QFN:DFN-6-1EP_3x3mm_P0.95mm_EP1.7x2.6mm, symbol REG1117A-1.8:REG1117A-1.8
- added IC2: REG1117A-2.5, Package_DFN_QFN:DFN-6-1EP_3x3mm_P0.95mm_EP1.7x2.6mm, symbol REG1117A-2.5:REG1117A-2.5
Connections:
- net 1V8: now also C1.1, IC1.2 (VOUT)
- net 2V5: now also C4.1, IC2.2 (VOUT)
- net 5V: now also C2.1, C3.1, IC1.3 (VIN), IC2.3 (VIN)
- net GND: now also C1.2, C2.2, C3.2, C4.2, IC1.1 (GND), IC2.1 (GND)
Other:
- moved on the sheet: TP1, TP2

Commit message: Fixed more issues
Connections:
- net 1V8 renamed +1V8
- net 2V5 renamed +2V5
- net 5V renamed +5V
Other:
- note added: "Reference for REG1117"
- note added: "Using tantalum capacitors"
- note removed: "Reference for LT1761-1.8"
