File: TX_ADAR/TX_ADAR.kicad_pcb (KiCad board)
At the start: 2 copper layers, 0 parts

Commit message: Adding to layout
Parts:
- added C1: 10uF, Capacitor_SMD:C_0603_1608Metric_Pad1.08x0.95mm_HandSolder, F.Cu at (256.9, 105.1)
- added C12: 100pF, Capacitor_SMD:C_0603_1608Metric_Pad1.08x0.95mm_HandSolder, F.Cu at (-47.5, 136.5)
- added C13: 100pF, Capacitor_SMD:C_0603_1608Metric_Pad1.08x0.95mm_HandSolder, F.Cu at (-47.5, 139.0)
- added C16: 10nF, Capacitor_SMD:C_0603_1608Metric_Pad1.08x0.95mm_HandSolder, F.Cu at (-47.5, 141.5)
- added C17: 100nF, Capacitor_SMD:C_0603_1608Metric_Pad1.08x0.95mm_HandSolder, F.Cu at (-70.9, 132.0)
- added C18: 100nF, Capacitor_SMD:C_0603_1608Metric_Pad1.08x0.95mm_HandSolder, F.Cu at (-70.9, 134.5)
- added C19: 100nF, Capacitor_SMD:C_0603_1608Metric_Pad1.08x0.95mm_HandSolder, F.Cu at (-70.9, 137.0)
- added C2: 10uF, Capacitor_SMD:C_0603_1608Metric_Pad1.08x0.95mm_HandSolder, F.Cu at (-54.1, 134.5)
- added C20: 100nF, Capacitor_SMD:C_0603_1608Metric_Pad1.08x0.95mm_HandSolder, F.Cu at (-70.9, 139.5)
- added C21: 100nF, Capacitor_SMD:C_0603_1608Metric_Pad1.08x0.95mm_HandSolder, F.Cu at (-70.9, 142.0)
- added C22: 100nF, Capacitor_SMD:C_0603_1608Metric_Pad1.08x0.95mm_HandSolder, F.Cu at (-66.5, 132.0)
- added C23: 100nF, Capacitor_SMD:C_0603_1608Metric_Pad1.08x0.95mm_HandSolder, F.Cu at (-66.5, 134.5)
- added C24: 100nF, Capacitor_SMD:C_0603_1608Metric_Pad1.08x0.95mm_HandSolder, F.Cu at (-66.5, 137.0)
- added C25: 100nF, Capacitor_SMD:C_0603_1608Metric_Pad1.08x0.95mm_HandSolder, F.Cu at (-66.5, 139.5)
- added C26: 100nF, Capacitor_SMD:C_0603_1608Metric_Pad1.08x0.95mm_HandSolder, F.Cu at (-66.5, 142.0)
- added C27: 100nF, Capacitor_SMD:C_0603_1608Metric_Pad1.08x0.95mm_HandSolder, F.Cu at (-62.2, 132.0)
- added C28: 100nF, Capacitor_SMD:C_0603_1608Metric_Pad1.08x0.95mm_HandSolder, F.Cu at (-62.2, 134.5)
- added C29: 100nF, Capacitor_SMD:C_0603_1608Metric_Pad1.08x0.95mm_HandSolder, F.Cu at (-31.4, 130.9)
- added C3: 10uF, Capacitor_SMD:C_0603_1608Metric_Pad1.08x0.95mm_HandSolder, F.Cu at (-54.1, 137.0)
- added C30: 100nF, Capacitor_SMD:C_0603_1608Metric_Pad1.08x0.95mm_HandSolder, F.Cu at (-31.4, 133.5)
- added C31: 100nF, Capacitor_SMD:C_0603_1608Metric_Pad1.08x0.95mm_HandSolder, F.Cu at (-31.4, 136.0)
- added C32: 1uF, Capacitor_SMD:C_0603_1608Metric_Pad1.08x0.95mm_HandSolder, F.Cu at (-43.1, 131.5)
- added C33: 10nF, Capacitor_SMD:C_0603_1608Metric_Pad1.08x0.95mm_HandSolder, F.Cu at (-43.1, 134.0)
- added C34: 10nF, Capacitor_SMD:C_0603_1608Metric_Pad1.08x0.95mm_HandSolder, F.Cu at (-43.1, 136.5)
- added C35: 100pF, Capacitor_SMD:C_0603_1608Metric_Pad1.08x0.95mm_HandSolder, F.Cu at (-43.1, 139.0)
- added C36: 10nF, Capacitor_SMD:C_0603_1608Metric_Pad1.08x0.95mm_HandSolder, F.Cu at (-43.1, 141.5)
- added C37: 100pF, Capacitor_SMD:C_0603_1608Metric_Pad1.08x0.95mm_HandSolder, F.Cu at (-38.8, 131.5)
- added C38: 100nF, Capacitor_SMD:C_0603_1608Metric_Pad1.08x0.95mm_HandSolder, F.Cu at (-31.4, 138.5)
- added C39: 100nF, Capacitor_SMD:C_0603_1608Metric_Pad1.08x0.95mm_HandSolder, F.Cu at (-31.4, 141.0)
- added C4: 10uF, Capacitor_SMD:C_0603_1608Metric_Pad1.08x0.95mm_HandSolder, F.Cu at (256.9, 85.1)
- added C40: 100nF, Capacitor_SMD:C_0603_1608Metric_Pad1.08x0.95mm_HandSolder, F.Cu at (-31.4, 143.5)
- added C41: 100nF, Capacitor_SMD:C_0603_1608Metric_Pad1.08x0.95mm_HandSolder, F.Cu at (123.0, 76.4)
- added C42: 100nF, Capacitor_SMD:C_0603_1608Metric_Pad1.08x0.95mm_HandSolder, F.Cu at (-18.0, 138.0)
- added C8: 100pF, Capacitor_SMD:C_0603_1608Metric_Pad1.08x0.95mm_HandSolder, F.Cu at (-47.5, 131.5)
- added C9: 1uF, Capacitor_SMD:C_0603_1608Metric_Pad1.08x0.95mm_HandSolder, F.Cu at (-47.5, 134.0)
- added H1: MountingHole_Pad, MountingHole:MountingHole_2.2mm_M2_DIN965_Pad, F.Cu at (19.0, 61.5)
- added H2: MountingHole_Pad, MountingHole:MountingHole_2.2mm_M2_DIN965_Pad, F.Cu at (19.0, 192.5)
- added H3: MountingHole_Pad, MountingHole:MountingHole_2.2mm_M2_DIN965_Pad, F.Cu at (281.0, 62.0)
- added H4: MountingHole_Pad, MountingHole:MountingHole_2.2mm_M2_DIN965_Pad, F.Cu at (281.5, 191.0)
- added IC1: REG1117A-1.8, REG1117A_1_8:SOT230P700X180-4N, F.Cu at (257.8, 97.6)
- added IC2: REG1117A-2.5, REG1117A_2_5:SOT230P700X180-4N, F.Cu at (257.8, 78.1)
- added J1: Conn_Coaxial, Connector_Coaxial:SMA_Amphenol_132289_EdgeMount, F.Cu at (278.6, 88.5)
- added J10: Conn_Coaxial, 142_1701_831:BEL_142-1701-831, F.Cu at (178.9, 29.0)
- added J11: RJ45_LED_Shielded, Connector_RJ:RJ45_Amphenol_RJHSE538X, F.Cu at (31.4, 106.7)
- added J12: RJ45_LED_Shielded, Connector_RJ:RJ45_Amphenol_RJHSE538X, F.Cu at (31.1, 139.2)
- added J15: FX8-120S-SV21, 120Conn footprints:CONN120_FX8-120S-SV_HIR, F.Cu at (278.4, 136.9)
- added J16: RJ45_LED_Shielded, Connector_RJ:RJ45_Amphenol_RJHSE538X, F.Cu at (31.0, 166.2)
- added J19: Conn_Coaxial, 142_1701_831:BEL_142-1701-831, F.Cu at (128.1, 232.9)
- added J2: Conn_Coaxial, 142_1701_831:BEL_142-1701-831, F.Cu at (77.8, 60.1)
- added J20: Conn_Coaxial, 142_1701_831:BEL_142-1701-831, F.Cu at (65.5, 232.8)
- added J21: Conn_01x04, Connector_PinHeader_2.54mm:PinHeader_1x04_P2.54mm_Vertical, F.Cu at (71.5, 158.2)
- added J3: Conn_Coaxial, 142_1701_831:BEL_142-1701-831, F.Cu at (116.3, 45.7)
- added J4: Conn_Coaxial, 142_1701_831:BEL_142-1701-831, F.Cu at (116.3, 29.0)
- added J5: Conn_Coaxial, 142_1701_831:BEL_142-1701-831, F.Cu at (123.4, 15.3)
- added J6: Conn_Coaxial, 142_1701_831:BEL_142-1701-831, F.Cu at (138.0, 15.3)
- added J7: Conn_Coaxial, 142_1701_831:BEL_142-1701-831, F.Cu at (171.3, 15.1)
- added J8: Conn_Coaxial, 142_1701_831:BEL_142-1701-831, F.Cu at (156.0, 15.1)
- added J9: Conn_Coaxial, 142_1701_831:BEL_142-1701-831, F.Cu at (178.9, 45.5)
- added R2: 50k, Resistor_SMD:R_0603_1608Metric_Pad0.98x0.95mm_HandSolder, F.Cu at (-62.2, 137.0)
- added R3: 50k, Resistor_SMD:R_0603_1608Metric_Pad0.98x0.95mm_HandSolder, F.Cu at (-62.2, 139.5)
- added R4: 50k, Resistor_SMD:R_0603_1608Metric_Pad0.98x0.95mm_HandSolder, F.Cu at (-18.0, 143.0)
- added R5: 50ohm, Resistor_SMD:R_0603_1608Metric_Pad0.98x0.95mm_HandSolder, F.Cu at (-38.8, 134.0)
- added R6: 50ohm, Resistor_SMD:R_0603_1608Metric_Pad0.98x0.95mm_HandSolder, F.Cu at (-38.8, 136.5)
- added SW1: SW_SPDT, 100SP1T1B4M2QE:SW_100SP1T1B4M2QE, F.Cu at (151.5, 118.5)
- added SW2: SW_SPDT, 100SP1T1B4M2QE:SW_100SP1T1B4M2QE, F.Cu at (238.0, 109.0)
- added SW3: SW_SPDT, 100SP1T1B4M2QE:SW_100SP1T1B4M2QE, F.Cu at (157.5, 74.5)
- added SW4: SW_SPDT, 100SP1T1B4M2QE:SW_100SP1T1B4M2QE, F.Cu at (151.0, 97.5)
- added SW9: SW_SPDT, 100SP1T1B4M2QE:SW_100SP1T1B4M2QE, F.Cu at (238.0, 88.5)
- added TP3: TestPoint, TestPoint:TestPoint_Loop_D2.50mm_Drill1.0mm, F.Cu at (221.5, 113.8)
- added TP4: TestPoint, TestPoint:TestPoint_Loop_D2.50mm_Drill1.0mm, F.Cu at (220.0, 93.0)
- added U10: TXB0101DBV, Package_TO_SOT_SMD:SOT-23-6, F.Cu at (-45.4, 81.3)
- added U11: TXB0101DBV, Package_TO_SOT_SMD:SOT-23-6, F.Cu at (-45.4, 85.9)
- added U12: TXB0101DBV, Package_TO_SOT_SMD:SOT-23-6, F.Cu at (-45.4, 90.5)
- added U13: TXB0101DBV, Package_TO_SOT_SMD:SOT-23-6, F.Cu at (134.1, 76.5)
- added U14: TXB0101DBV, Package_TO_SOT_SMD:SOT-23-6, F.Cu at (-39.1, 86.0)
- added U15: TXB0101DBV, Package_TO_SOT_SMD:SOT-23-6, F.Cu at (-17.2, 170.9)
- added U16: TXB0101DBV, Package_TO_SOT_SMD:SOT-23-6, F.Cu at (-17.0, 179.1)
- added U17: TXB0101DBV, Package_TO_SOT_SMD:SOT-23-6, F.Cu at (-17.1, 186.1)
- added U18: TXB0101DBV, Package_TO_SOT_SMD:SOT-23-6, F.Cu at (-17.0, 193.5)
- added U19: TXB0101DBV, Package_TO_SOT_SMD:SOT-23-6, F.Cu at (-39.1, 90.6)
- added U2: ADAR2001ACCZ, ADAR footprints:LGA-CC-40-7_ADI, F.Cu at (147.5, 37.2)
Other:
- board text added: "Cal Line"
- board text added: "RF Out"
- board text added: "The star is bttm left"
- board text removed: "External"
- board text removed: "Level Shifters"
- board text removed: "RF In and Out"
- board text removed: "SPI Comms Level Shifters"

Commit message: Layout changes
Parts:
- moved C3 330.2 mm to (271.5, 82.5), turned to 90 degrees
- moved C2 328.1 mm to (272.0, 98.6), turned to -90 degrees
- moved H4 320.8 mm to (-15.0, 68.5)
- moved H3 297.2 mm to (-16.0, 50.5)
- moved H2 137.4 mm to (-15.5, 59.5)
- moved J2 55.0 mm to (116.4, 21.0), turned to 90 degrees
- moved J10 46.0 mm to (179.0, -17.1)
- moved J3 46.0 mm to (116.4, -0.31)
- moved J6 46.0 mm to (138.2, -30.8)
- moved J8 46.0 mm to (156.1, -31.0)
- moved J4 46.0 mm to (116.5, -17.0)
- moved J5 46.0 mm to (123.6, -30.8)
- moved J7 46.0 mm to (171.5, -30.9)
- moved J9 46.0 mm to (179.1, -0.53)
- moved U2 46.0 mm to (147.7, -8.84)
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Routing:
- net +5V: track 0.00 -> 23.8 mm
Other:
- copper layers 2 -> 4
- board text added: "Out1+"
- board text added: "Out1-"
- board text added: "Out2+"
- board text added: "Out2-"
- board text added: "Out3+"
- board text added: "Out3-"
- board text added: "Out4+"
- board text added: "Out4-"
- board text added: "RF In"

Commit message: Layout Editting
Lots to move around
Parts:
- moved J16 251.9 mm to (273.5, 97.9), turned to -90 degrees
- moved C9 237.9 mm to (150.5, 2.00)
- moved C8 234.2 mm to (150.6, 6.50)
- moved C33 232.0 mm to (156.1, 15.0)
- moved C12 229.4 mm to (149.9, 19.5)
- moved C34 228.1 mm to (149.9, 15.0)
- moved C36 225.5 mm to (143.5, 15.0)
- moved C32 225.1 mm to (181.6, 143.5)
- moved C37 224.6 mm to (155.9, 19.5)
- moved C16 224.4 mm to (137.9, 15.0)
- moved J21 223.1 mm to (278.5, 74.9)
- moved C35 221.6 mm to (143.5, 19.5)
- moved C13 220.5 mm to (137.9, 19.5)
- moved R3 203.9 mm to (139.4, 108.5)
- moved C30 176.4 mm to (120.4, 43.5)
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Routing:
- net +5V: track 23.8 -> 0.00 mm
Other:
- board text added: "Thru Cal Line Length = 2 x RF Output"
- board text added: "TxADV TxRST MADV MRST"
- board text removed: "ADAR"
- board text removed: "Cal Line"
- board text removed: "Power Delivery"
- board text removed: "RF Out"
- board text removed: "The star is bttm left"

Commit message: Progress on layout
Rough idea of where each component will be relative to each other.
Had some ideas about a component that might be redundant.
Need to determine the final orientation of the components and size of pcb.
Parts:
- moved H4 299.9 mm to (244.5, 164.5)
- moved H3 287.8 mm to (244.5, 15.5)
- moved R2 287.6 mm to (229.0, 78.5), turned to 90 degrees
- moved C20 284.4 mm to (209.6, 97.5)
- moved C25 282.1 mm to (209.5, 86.0)
- moved C26 275.5 mm to (194.6, 63.0), turned to 180 degrees
- moved C18 274.4 mm to (209.4, 91.5)
- moved C21 271.4 mm to (195.0, 97.6), turned to 180 degrees
- moved C24 268.1 mm to (209.6, 104.0)
- moved C22 267.5 mm to (209.9, 116.5)
- moved C28 263.3 mm to (209.6, 110.5)
- moved C17 262.9 mm to (194.6, 74.5), turned to 180 degrees
- moved C42 258.8 mm to (209.1, 69.0)
- moved C19 256.8 mm to (195.5, 116.4), turned to 180 degrees
- moved C23 253.5 mm to (195.3, 110.4), turned to 180 degrees
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Connections:
- SW3 pad 2: /CSB -> /External Input/3V3CSB
- U10 pad 3: /External Input/3V3_SDIO -> /SDIO
- U10 pad 4: /SDIO -> /External Input/3V3_SDIO
- U11 pad 3: /External Input/3V3SDO -> /SDO
- U11 pad 4: /SDO -> /External Input/3V3SDO
- U12 pad 3: /External Input/3V3SDIO2 -> /SPI Communications/1V8SDIO2
- U12 pad 4: /SPI Communications/1V8SDIO2 -> /External Input/3V3SDIO2
- U13 pad 3: /External Input/3V3SDIO3 -> /SPI Communications/1V8SDIO3
- U13 pad 4: /SPI Communications/1V8SDIO3 -> /External Input/3V3SDIO3
- U14 pad 3: /External Input/3V3CSB -> /CSB
- U14 pad 4: /CSB -> /External Input/3V3CSB
- U15 pad 3: /External Input/TxADV -> /TxADV
- U15 pad 4: /TxADV -> /External Input/TxADV
- U16 pad 3: /External Input/TxRST -> /TxRST
- U16 pad 4: /TxRST -> /External Input/TxRST
- U17 pad 3: /External Input/MADV -> /MADV
- U17 pad 4: /MADV -> /External Input/MADV
- U18 pad 3: /External Input/MRST -> /MRST
- U18 pad 4: /MRST -> /External Input/MRST
- U19 pad 3: /External Input/3V3_SCLK -> /SCLK
- U19 pad 4: /SCLK -> /External Input/3V3_SCLK
Other:
- board outline added: 98.8 x 276.1 mm
- board text added: "Make ic pin longer"

Commit message: Layout Updates
Parts:
- removed R4: 50k, Resistor_SMD:R_0603_1608Metric_Pad0.98x0.95mm_HandSolder
- removed SW4: SW_SPDT, 100SP1T1B4M2QE:SW_100SP1T1B4M2QE
- moved J12 149.1 mm to (98.0, 126.5), turned to 90 degrees
- moved J11 122.5 mm to (126.9, 136.4), turned to 180 degrees
- moved J16 120.4 mm to (97.7, 56.5), turned to 90 degrees
- moved TP4 119.4 mm to (199.5, 138.0), turned to 0 degrees
- moved J1 108.9 mm to (177.9, 142.8), turned to -90 degrees
- moved J21 102.8 mm to (109.8, 49.0), turned to 0 degrees
- moved TP3 99.3 mm to (155.5, 137.8), turned to 0 degrees
- moved C2 99.2 mm to (182.6, 135.5), turned to 0 degrees
- moved C22 99.1 mm to (126.8, 62.3), turned to 180 degrees
- moved C24 99.0 mm to (127.1, 49.5), turned to 180 degrees
- moved C20 98.9 mm to (127.4, 42.5), turned to 180 degrees
- moved C3 98.9 mm to (173.5, 135.5), turned to 180 degrees
- moved C28 98.9 mm to (127.2, 55.9), turned to 180 degrees
- moved R2 91.2 mm to (148.5, 121.3)
- moved SW1 91.2 mm to (142.5, 115.8)
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Connections:
- U15 pad 5: /Sequencer Level Shifter/OE -> /SPI Communications/OE
- U16 pad 5: /Sequencer Level Shifter/OE -> /SPI Communications/OE
- U17 pad 5: /Sequencer Level Shifter/OE -> /SPI Communications/OE
- U18 pad 5: /Sequencer Level Shifter/OE -> /SPI Communications/OE
Routing:
- net +1V8: track 0.00 -> 68.3 mm
- net /External Input/3V3_VCCB_SPI: track 0.00 -> 43.6 mm
- net /External Input/TxADV: track 0.00 -> 36.5 mm
- net +2V5: track 0.00 -> 35.6 mm
- net /External Input/MRST: track 0.00 -> 35.0 mm
- net +5V: track 0.00 -> 34.5 mm
- net /External Input/TxRST: track 0.00 -> 34.5 mm
- net /External Input/MADV: track 0.00 -> 33.4 mm
- net Net-(IC2-VOUT): track 0.00 -> 17.9 mm
- net Net-(IC1-VOUT): track 0.00 -> 13.4 mm
- net Net-(SW9-A): track 0.00 -> 9.00 mm
- net Net-(SW2-A): track 0.00 -> 8.11 mm
- net Net-(SW1-A): track 0.00 -> 6.05 mm
- net /TxADV: track 0.00 -> 5.81 mm
- net Net-(SW3-A): track 0.00 -> 4.39 mm
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Other:
- board size 98.8 x 276.1 mm -> 130 x 275.3 mm
- board text added: "Might be best to push 2V5 to boundary at the top"

Commit message: Layout comments and slight changes
Parts:
- moved J19 89.1 mm to (118.4, 179.9)
- moved J20 89.1 mm to (25.5, 180.1)
- moved SW3 40.0 mm to (143.5, 135.7), turned to 0 degrees
- moved R3 23.3 mm to (143.5, 125.7), turned to 90 degrees
- moved C17 6.75 mm to (141.2, 69.0)
- moved C40 6.75 mm to (127.6, 69.0)
- moved U11 6.75 mm to (134.0, 68.0)
- moved C39 6.21 mm to (141.1, 75.5)
- moved U19 6.21 mm to (133.9, 74.5)
- moved C42 6.21 mm to (127.7, 75.5)
- moved R2 2.24 mm to (149.5, 119.3)
- moved SW1 1.80 mm to (143.5, 114.3)
Routing:
- net +1V8: track 68.3 -> 74.4 mm
Other:
- board size 130 x 275.3 mm -> 190.4 x 230.7 mm
- board text added: "3V3 comes in from right 1V8 comes in from left OE goes in from right Level shifter out goes out from left"
- board text added: "Add baluns?"
- board text added: "Add more space for RF In for better isolation?"
- board text added: "Close enough to edge?"
- board text added: "Connectors too close to each other? Too close to the other pair?"
- board text added: "Do we even need this on the same PCB?"
- board text added: "Easier to work with vias with 120 pin in middle"
- board text added: "For 3V3 connection of switch: Via to bttm and connect to copper fill area"
- board text added: "Good distance away?"
- board text added: "Make ic pin longer & simulate(?)"
- board text added: "Might be best to push 2V5 to boundary at the top bc it goes into ADAR"
- board text added: "Need to connect these two pieces so traces can go through"
- board text added: "Use tantalum capacitors"
- board text removed: "Make ic pin longer"
- board text removed: "Might be best to push 2V5 to boundary at the top"

Commit message: Got layout feedback from flatrim
Parts:
- removed C26: 100nF, Capacitor_SMD:C_0603_1608Metric_Pad1.08x0.95mm_HandSolder
- removed J15: FX8-120S-SV21, 120Conn footprints:CONN120_FX8-120S-SV_HIR
- removed J19, J20: Conn_Coaxial, 142_1701_831:BEL_142-1701-831
- removed U12, U13: TXB0101DBV, Package_TO_SOT_SMD:SOT-23-6
- moved H1 233.3 mm to (306.5, 119.0)
- moved H2 213.7 mm to (299.5, 119.0)
- moved C41 169.7 mm to (1.68, 5.78)
- moved C38 160.4 mm to (1.68, 3.27), turned to 0 degrees
- moved C30 158.1 mm to (1.68, 0.76), turned to 0 degrees
- moved H3 132.5 mm to (315.0, 120.0)
- moved H4 115.4 mm to (322.5, 121.0)
- moved TP4 102.0 mm to (102.6, 106.0), turned to -90 degrees
- moved C2 90.3 mm to (105.1, 89.1), turned to -90 degrees
- moved SW9 85.2 mm to (116.3, 106.0), turned to 90 degrees
- moved C20 83.4 mm to (205.4, 72.0), turned to 0 degrees
- moved C4 81.8 mm to (115.4, 99.5), turned to 180 degrees
- moved C24 80.2 mm to (205.7, 65.0), turned to 0 degrees
- moved C22 79.7 mm to (205.9, 52.1), turned to 0 degrees
- moved IC2 79.4 mm to (113.5, 90.5), turned to 0 degrees
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Routing:
- net +1V8: track 74.4 -> 23.7 mm
- net /External Input/3V3_VCCB_SPI: track 43.6 -> 0.21 mm
- net /External Input/TxADV: track 36.5 -> 0.00 mm
- net /External Input/MRST: track 35.0 -> 0.00 mm
- net +5V: track 34.5 -> 0.00 mm
- net /External Input/TxRST: track 34.5 -> 0.00 mm
- net /External Input/MADV: track 33.4 -> 0.00 mm
- net /RFOut3-: track 0.00 -> 31.0 mm
- net /RFOut2-: track 0.00 -> 31.0 mm
- net +2V5: track 35.6 -> 16.7 mm
- net Net-(IC2-VOUT): track 17.9 -> 6.52 mm
- net Net-(SW9-A): track 9.00 -> 0.00 mm
Other:
- board size 190.4 x 230.7 mm -> 68.5 x 197.6 mm
- board text added: "MRST MADV TxRST TxADV"
- board text removed: "3V3 comes in from right 1V8 comes in from left OE goes in from right Level shifter out goes out from left"
- board text removed: "Add more space for RF In for better isolation?"
- board text removed: "Close enough to edge?"
- board text removed: "Connectors too close to each other? Too close to the other pair?"
- board text removed: "Do we even need this on the same PCB?"
- board text removed: "Easier to work with vias with 120 pin in middle"
- board text removed: "For 3V3 connection of switch: Via to bttm and connect to copper fill area"
- board text removed: "Might be best to push 2V5 to boundary at the top bc it goes into ADAR"
- board text removed: "Need to connect these two pieces so traces can go through"
- board text removed: "Thru Cal Line Length = 2 x RF Output"
- board text removed: "TxADV TxRST MADV MRST"
