File: TX_ADAR/TX_ADAR.kicad_pcb (KiCad board)
At the start: 4 copper layers, 68.5 x 197.6 mm, 73 parts, among them IC1 REG1117A-1.8, IC2 REG1117A-2.5, J1 Screw_Terminal_01x02, J10 Conn_Coaxial, J11 RJ45_LED_Shielded, J12 RJ45_LED_Shielded, J16 RJ45_LED_Shielded, J2 Conn_Coaxial, J21 Conn_01x04, J3 Conn_Coaxial, J4 Conn_Coaxial, J5 Conn_Coaxial, J6 Conn_Coaxial, J7 Conn_Coaxial, J8 Conn_Coaxial, J9 Conn_Coaxial, SW1 SW_SPDT, SW2 SW_SPDT, SW3 SW_SPDT, SW9 SW_SPDT, U10 TXB0101DBV, U11 TXB0101DBV, U14 TXB0101DBV, U15 TXB0101DBV, U16 TXB0101DBV, U17 TXB0101DBV, U18 TXB0101DBV, U19 TXB0101DBV, U2 ADAR2001ACCZ

Commit message: Layout moved, connectors lined up
Parts:
- moved H3 231.2 mm to (93.0, 184.5)
- moved H1 229.6 mm to (93.0, 34.5)
- moved H4 180.1 mm to (154.0, 184.5)
- moved H2 168.3 mm to (154.0, 34.5)
- moved C30 67.8 mm to (43.6, 54.0)
- moved C38 67.8 mm to (43.6, 56.5)
- moved C41 67.8 mm to (43.6, 59.0)
- moved R6 49.0 mm to (125.1, 76.5), turned to 0 degrees
- moved C17 48.6 mm to (134.7, 84.6)
- moved C25 48.6 mm to (140.5, 94.7)
- moved C31 48.6 mm to (134.7, 89.7)
- moved C39 48.6 mm to (134.8, 99.6)
- moved C40 48.6 mm to (140.5, 84.6)
- moved C42 48.6 mm to (140.5, 99.6)
- moved U10 48.6 mm to (137.6, 96.5)
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Routing:
- net +1V8: track 8.10 -> 15.1 mm
- net /External Input/3V3_VCCB_SPI: track 0.21 -> 7.14 mm
- net +2V5: track 12.3 -> 15.8 mm
Other:
- board size 68.5 x 197.6 mm -> 68 x 156.9 mm
- board text added: "Some may have to go to the bttm"

Commit message: Footprint updates
Parts:
- removed C19, C20, C21, C22, C23, C24, C27, C28, C30, C38, C41: 100nF, Capacitor_SMD:C_0603_1608Metric_Pad1.08x0.95mm_HandSolder
- removed U15, U16, U17, U18: TXB0101DBV, Package_TO_SOT_SMD:SOT-23-6
- J10, J2, J3, J4, J5, J6, J7, J8, J9: footprint 142_1701_831:BEL_142-1701-831 -> CON292001_1:TE_CON292001-1
- moved C29 17.4 mm to (150.9, 88.1), turned to 0 degrees
- moved C39 14.5 mm to (143.7, 88.2), turned to 0 degrees
- moved U10 12.7 mm to (149.1, 91.0), turned to -90 degrees
- moved C18 12.6 mm to (128.6, 93.9), turned to 0 degrees
- moved U19 11.2 mm to (141.9, 91.0), turned to -90 degrees
- moved U14 10.8 mm to (126.8, 91.0), turned to -90 degrees
- moved C25 10.5 mm to (150.9, 93.9), turned to 0 degrees
- moved C40 10.1 mm to (136.4, 93.9), turned to 0 degrees
- moved C42 6.56 mm to (143.7, 93.9), turned to 0 degrees
- moved C31 6.31 mm to (128.6, 88.2), turned to 0 degrees
- moved U11 5.46 mm to (134.6, 91.0), turned to -90 degrees
- moved J10 4.60 mm to (151.0, 58.7), turned to 0 degrees
- moved J9 4.51 mm to (150.7, 75.5), turned to 0 degrees
- moved C35 4.11 mm to (116.8, 56.0)
- moved C36 4.11 mm to (116.8, 54.5)
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Routing:
- net /External Input/3V3SDO: track 0.00 -> 33.9 mm
- net /RFOut1-: track 30.7 -> 0.01 mm
- net /RFOut2-: track 30.6 -> 0.00 mm
- net /RFOut4-: track 30.6 -> 0.01 mm
- net /RFOut3-: track 30.6 -> 0.00 mm
- net /External Input/3V3_SCLK: track 0.00 -> 28.8 mm
- net /External Input/3V3CSB: track 0.00 -> 28.1 mm
- net /External Input/3V3_SDIO: track 0.00 -> 27.7 mm
- net /SPI Communications/OE: track 0.00 -> 25.0 mm
- net /External Input/TxADV: track 0.00 -> 13.2 mm
- net /External Input/MRST: track 0.00 -> 12.8 mm
- net /External Input/MADV: track 0.00 -> 12.6 mm
- net /External Input/TxRST: track 0.00 -> 12.4 mm
- net +1V8: track 15.1 -> 22.7 mm
- net Net-(SW3-A): track 0.00 -> 7.21 mm
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Other:
- board text removed: "Add baluns?"
- board text removed: "Out1+"
- board text removed: "Out1-"
- board text removed: "Out2+"
- board text removed: "Out2-"
- board text removed: "Out3+"
- board text removed: "Out3-"
- board text removed: "Out4+"
- board text removed: "Out4-"
- board text removed: "RF In"

Commit message: Layout updates
Using vias to connect hard to reach spots
Added copper pours
Parts:
- added C19: 100nF, Capacitor_SMD:C_0603_1608Metric_Pad1.08x0.95mm_HandSolder, F.Cu at (28.7, 21.8)
- added C20: 100nF, Capacitor_SMD:C_0603_1608Metric_Pad1.08x0.95mm_HandSolder, F.Cu at (28.7, 24.3)
- added C21: 100nF, Capacitor_SMD:C_0603_1608Metric_Pad1.08x0.95mm_HandSolder, F.Cu at (28.7, 26.8)
- added C22: 100nF, Capacitor_SMD:C_0603_1608Metric_Pad1.08x0.95mm_HandSolder, F.Cu at (28.7, 29.3)
- added C27: 100nF, Capacitor_SMD:C_0603_1608Metric_Pad1.08x0.95mm_HandSolder, F.Cu at (28.7, 31.8)
- added C28: 100nF, Capacitor_SMD:C_0603_1608Metric_Pad1.08x0.95mm_HandSolder, F.Cu at (28.7, 34.3)
- added C30: 100nF, Capacitor_SMD:C_0603_1608Metric_Pad1.08x0.95mm_HandSolder, F.Cu at (22.3, 21.8)
- added C38: 100nF, Capacitor_SMD:C_0603_1608Metric_Pad1.08x0.95mm_HandSolder, F.Cu at (22.3, 24.3)
- added C41: 100nF, Capacitor_SMD:C_0603_1608Metric_Pad1.08x0.95mm_HandSolder, F.Cu at (22.3, 26.8)
- added U15: TXB0101DBV, Package_TO_SOT_SMD:SOT-23-6, F.Cu at (17.6, 22.9)
- added U16: TXB0101DBV, Package_TO_SOT_SMD:SOT-23-6, F.Cu at (17.6, 27.5)
- added U17: TXB0101DBV, Package_TO_SOT_SMD:SOT-23-6, F.Cu at (17.6, 32.1)
- added U18: TXB0101DBV, Package_TO_SOT_SMD:SOT-23-6, F.Cu at (17.6, 36.8)
- moved C29 16.9 mm to (134.0, 89.0)
- moved C39 16.9 mm to (126.9, 89.0)
- moved C42 16.9 mm to (126.9, 94.7)
- moved U19 16.9 mm to (125.0, 91.9)
- moved C25 16.9 mm to (134.0, 94.7)
- moved U10 16.9 mm to (132.2, 91.9)
- moved U14 12.9 mm to (139.7, 91.9)
- moved C18 12.9 mm to (141.5, 94.7)
- moved C31 12.9 mm to (141.5, 89.0)
- moved U11 12.7 mm to (147.3, 91.8)
- moved C17 12.7 mm to (149.1, 88.9)
- moved C40 12.7 mm to (149.1, 94.7)
- moved SW3 2.82 mm to (122.0, 178.5)
- moved J5 2.50 mm to (102.0, 34.0)
- moved J6 2.50 mm to (115.0, 34.0)
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Routing:
- net +1V8: track 22.7 -> 108.1 mm, vias 0 -> 5
- net /External Input/3V3_VCCB_SPI: track 6.93 -> 85.0 mm, vias 0 -> 4
- net /SPI Communications/OE: track 25.0 -> 92.2 mm, vias 0 -> 4
- net /External Input/3V3SDO: track 33.9 -> 0.00 mm
- net /RFOut4-: track 0.01 -> 26.2 mm
- net /RFOut3-: track 0.00 -> 26.1 mm
- net /RFOut1-: track 0.01 -> 26.1 mm
- net /RFOut2-: track 0.00 -> 26.0 mm
- net /External Input/3V3_SCLK: track 28.8 -> 35.6 mm
- net /External Input/3V3_SDIO: track 27.7 -> 31.3 mm
- net +2V5: track 21.3 -> 24.3 mm, vias 0 -> 1
- net Net-(SW3-A): track 7.21 -> 5.56 mm
- net /External Input/3V3CSB: track 28.1 -> 29.7 mm
- net Net-(IC1-VOUT): track 14.7 -> 13.6 mm
- added copper zone on B.Cu, net +1V8
- added copper zone on B.Cu, net /External Input/3V3_VCCB_SPI
- added copper zone on B.Cu, net /SPI Communications/OE
Other:
- board text added: "50 ohm term Use resistor to breach connector pin and gnd"
- board text added: "Out1+"
- board text added: "Out1-"
- board text added: "Out2+"
- board text added: "Out2-"
- board text added: "Out3+"
- board text added: "Out3-"
- board text added: "Out4+"
- board text added: "Out4-"
- board text added: "RF In"

Commit message: Updates to layout and connectors
**Need to add 50 ohm term to gnd from connector on positive outs for 2.92 vert launches**
Parts:
- removed C19, C20, C21, C22, C27, C28, C30, C38, C41: 100nF, Capacitor_SMD:C_0603_1608Metric_Pad1.08x0.95mm_HandSolder
- removed U15, U16, U17, U18: TXB0101DBV, Package_TO_SOT_SMD:SOT-23-6
- C12, C13, C16, C33, C34, C35, C36, C37, C8, C9: moved to B.Cu
- moved R6 8.82 mm to (125.9, 65.5)
- moved R5 8.51 mm to (123.9, 67.0)
- moved J3 5.02 mm to (97.5, 71.0)
- moved J9 5.00 mm to (147.7, 71.5)
- moved J2 4.00 mm to (97.5, 89.9)
- moved J4 4.00 mm to (97.3, 58.7)
- moved C8 4.00 mm to (123.4, 64.5)
- moved J8 3.16 mm to (128.4, 37.0)
- moved J7 3.16 mm to (141.0, 37.0)
- moved J10 3.02 mm to (147.9, 58.7)
- moved J5 3.00 mm to (102.0, 37.0)
- moved J6 3.00 mm to (115.0, 37.0)
- moved C33 2.52 mm to (127.1, 57.0)
- moved C36 2.52 mm to (117.1, 57.0)
- moved C34 2.38 mm to (117.2, 63.8)
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Connections:
- J10 pad 4: (no net) -> GND
- J3 pad 4: (no net) -> GND
- J4 pad 4: (no net) -> GND
- J5 pad 4: (no net) -> GND
- J6 pad 4: (no net) -> GND
- J7 pad 4: (no net) -> GND
- J8 pad 4: (no net) -> GND
- J9 pad 4: (no net) -> GND
Routing:
- net /External Input/3V3CSB: track 29.7 -> 103.9 mm, vias 0 -> 1
- net +2V5: track 24.3 -> 73.7 mm, vias 1 -> 5
- net /SDO: track 0.00 -> 39.3 mm
- net /CSB: track 0.00 -> 35.6 mm
- net /SDIO: track 0.00 -> 32.0 mm
- net /SCLK: track 0.00 -> 31.4 mm
- net /External Input/3V3SDO: track 0.00 -> 30.5 mm, vias 0 -> 1
- net /RFOut4-: track 26.2 -> 0.08 mm
- net /RFOut3-: track 26.1 -> 0.00 mm
- net /RFOut1-: track 26.1 -> 0.01 mm
- net /RFOut2-: track 26.0 -> 0.00 mm
- net +1V8: track 108.1 -> 130.6 mm, vias 5 -> 6
- net /External Input/3V3_VCCB_SPI: track 85.0 -> 86.2 mm
- added copper zone on B.Cu, net +2V5
Other:
- board text added: "+1V8"
- board text added: "+2V5"
- board text added: "+3V3"
- board text added: "OE"
- board text removed: "Make ic pin longer & simulate(?)"
- board text removed: "Some may have to go to the bttm"

Commit message: Layout Update
Routing:
- net /RFIN: track 0.00 -> 43.0 mm
