File: TX_ADAR/_restore_backup_2026-09-08T10-13-37-232/Connectors.kicad_sch (KiCad schematic)
At the start: 10 parts, among them J1 Conn_Coaxial, J11 RJ45_LED_Shielded, J12 RJ45_LED_Shielded, J13 Conn_Coaxial, J14 Conn_Coaxial, J15 FX8-120S-SV21, J16 RJ45_LED_Shielded, J17 Conn_Coaxial, J18 Conn_Coaxial, J2 Conn_Coaxial

Commit message: Some footprints updated and power buffers added
Parts:
- J2: footprint (none) -> Connector_Coaxial:SMA_Amphenol_132289_EdgeMount
Changed lines of the file:
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@@
 			)
 		)
-		(property "Footprint" ""
+		(property "Footprint" "Connector_Coaxial:SMA_Amphenol_132289_EdgeMount"
 			(at 57.15 19.05 0)
 			(hide yes)
