File: AD9248/ADC_unit.kicad_sch (KiCad schematic)
At the start: 37 parts, among them U1 TLV70018DCKR, U10 TXB0101DBVR, U11 DS90LV048ATMX/NOPB, U12 DS90LV048ATMX/NOPB, U2 AD9284BCPZ-250, U3 TLV70018DCKR, U8 TXB0101DBVR, U9 TXB0101DBVR

Commit message: Schematic under construction - clock / analog input driver defered but digital outputs are now wired correctly with correct differential impedance
Parts:
- added C24, C30, C31: GRM188R60J106ME47D, part_library:GRM188R60J106ME47D, symbol GRM188R60J106ME47D:GRM188R60J106ME47D
- added C25: GCM188R71E105KA64D, part_library:GCM188R71E105KA64D, symbol GCM188R71E105KA64D:GCM188R71E105KA64D
- added C26, C27, C33, C34: C0603C104K5RACTU, part_library:C0603C104K5RACTU, symbol C0603C104K5RACTU:C0603C104K5RACTU
- added C28, C29, C32: C0603C102K5RACTU, part_library:C0603C102K5RACTU, symbol C0603C102K5RACTU:C0603C102K5RACTU
- added R11, R13, R15, R17, R19, R21, R23, R5, R9: RMCF1206FG100R, part_library:RMCF1206FG100R, symbol RMCF1206FG100R:RMCF1206FG100R
- added U5: DS90LV048ATMX/NOPB, part_library:SOIC16, symbol DS9:DS90LV048ATMX_NOPB
- added U7: ADA4937-1YCPZ-R7, part_library:ADA4937_1YCPZ_R7, symbol ADA4937_1YCPZ_R7:ADA4937-1YCPZ-R7
Connections:
- net GND: now also C24.1, C25.1, C26.1, C27.1, C28.1, C29.1, C30.1, C31.1, C32.1, C33.1, C34.1, U5.12 (GND), U5.9 (~EN)
- net VCC_Analog: now also C30.2
- net VCC_Digital: now also C31.2; no longer U12.13 (VCC), U12.16 (EN)
- net VCC_Raw: now also U12.13 (VCC), U12.16 (EN), C24.2, C25.2, C26.2, C27.2, C28.2, C29.2, C32.2, C33.2, U5.13 (VCC), U5.16 (EN)
- net VREF: now also C34.2
- net at U12.1 (RIN1-), U2.25 (D7-(MSB)): now also R23.2
- net at U12.2 (RIN1+), U2.26 (D7+(MSB)): now also R23.1
- net at U12.3 (RIN2+), U2.24 (D6+): now also R21.1
- net at U12.4 (RIN2-), U2.23 (D6-): now also R21.2
- net at U12.5 (RIN3-), U2.21 (D5-): now also R19.2
- net at U12.6 (RIN3+), U2.22 (D5+): now also R19.1
- net at U12.7 (RIN4+), U2.20 (D4+): now also R17.1
- net at U12.8 (RIN4-), U2.19 (D4-): now also R17.2
- net at U2.10 (D0+(LSB)): now also U11.7 (RIN4+), R5.1
- net at U2.11 (D1-): now also U11.5 (RIN3-), R9.2; no longer U11.8 (RIN4-)
- net at U2.12 (D1+): now also U11.6 (RIN3+), R9.1; no longer U11.7 (RIN4+)
- net at U2.13 (D2-): now also U11.4 (RIN2-), R11.2; no longer U11.5 (RIN3-)
- net at U2.14 (D2+): now also U11.3 (RIN2+), R11.1; no longer U11.6 (RIN3+)
- net at U2.15 (D3-): now also U11.1 (RIN1-), R13.2; no longer U11.4 (RIN2-)
- net at U2.16 (D3+): now also U11.2 (RIN1+), R13.1; no longer U11.3 (RIN2+)
- net at U2.17 (DCO-): now also R15.2, U5.8 (RIN4-); no longer U11.1 (RIN1-)
- net at U2.18 (DCO+): now also R15.1, U5.7 (RIN4+); no longer U11.2 (RIN1+)
- net at U2.9 (D0-(LSB)): now also U11.8 (RIN4-), R5.2
- net CSB: no longer names the net of U2.32 (CSB), U8.3 (A)
- net SCLK: no longer names the net of U2.30 (SCLK), U9.3 (A)
- net SDIO: no longer names the net of U10.3 (A), U2.31 (SDIO/PWDN)
- new net ADC_CLKOUT: U5.10 (ROUT4)
Other:
- note added: "0.001u"
- note added: "100 ohm"
- note added: "10k"
- note added: "10uF"
- note added: "AD9248 BYPASS AND DECOUPLING"
- note added: "ADC"
- note added: "Mandatory 100 ohm differential impedance prior to reciever input"
- note added: "Note: MOSI needs to be pulled low post configuration, and CSB/NSS should be held high CLK should be inactive"
- note added: "SPI input and level shifting"
- note added: "[1] Pg. 17"
- note added: "[1] Pg. 22"
- note added: "[4] Pg. 12"
- note added: "[4] Pg. 13"
- note added: "[4] Pg. 3"
- note added: "[5] Pg. 14"
- note removed: "*TODO Note: we may need to add a .1uF pair to each of these (see eval board schematic), but we're running slower speeds so I'm just placing 1 for now"
- note removed: "ADC and digital conversion"
- note removed: "Decouplers"
- note removed: "LDOs"
- note removed: "SPI level shifting"
- moved on the sheet: C1, C10, C11, C12, C13, C14, C15, C16, C17, C18, C19, C2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

Commit message: Rough draft completete, TODO: Cosmetic stuff (Make it more modular in schematic), simulate sallen key with non-ideal components, check FPGA pinout constraints for clock generation, validate design
Parts:
- removed C1, C10, C2, C25, C3: GCM188R71E105KA64D, part_library:GCM188R71E105KA64D, symbol GCM188R71E105KA64D:GCM188R71E105KA64D
- removed C11, C16, C17, C20, C21, C22, C34, C4, C5, C6, C7, C8, C9: C0603C104K5RACTU, part_library:C0603C104K5RACTU, symbol C0603C104K5RACTU:C0603C104K5RACTU
- removed C12, C13, C14, C15, C18, C19: GRM3195C1H104JA05D, part_library:GRM3195C1H104JA05D, symbol GRM3195C1H104JA05D:GRM3195C1H104JA05D
- removed C24, C30, C31: GRM188R60J106ME47D, part_library:GRM188R60J106ME47D, symbol GRM188R60J106ME47D:GRM188R60J106ME47D
- removed R2, R3, R4, R7, R8: RC1206FR-0733RL, part_library:RC1206FR_0733RL, symbol RC1206FR_0733RL:RC1206FR-0733RL
- removed U1, U3: TLV70018DCKR, part_library:TLV70018DCKR, symbol TLV70018DCKR:TLV70018DCKR
- removed U10, U8, U9: TXB0101DBVR, part_library:TXB0101DBVR, symbol TXB0101DBVR:TXB0101DBVR
- removed U7: ADA4937-1YCPZ-R7, part_library:ADA4937_1YCPZ_R7, symbol ADA4937_1YCPZ_R7:ADA4937-1YCPZ-R7
- added C24: C0603C102K5RACTU, part_library:C0603C102K5RACTU, symbol C0603C102K5RACTU:C0603C102K5RACTU
- added C28, C29, C30, C31, C35, C36, C37, C38, C39, C40: C0603C104K5RACTU, part_library:C0603C104K5RACTU, symbol C0603C104K5RACTU:C0603C104K5RACTU
- added C41, C42: 06031AR47CAT2A, part_library:06031AR47CAT2A, symbol 06031AR47CAT2A:06031AR47CAT2A
- added R11: RMCF1206FG100R, part_library:RMCF1206FG100R, symbol RMCF1206FG100R:RMCF1206FG100R
- added R12, R13, R14, R15: RC1206FR-0733RL, part_library:RC1206FR_0733RL, symbol RC1206FR_0733RL:RC1206FR-0733RL
- added U13: DS90LV011ATMF/NOPB, Package_TO_SOT_SMD:SOT-23-5_HandSoldering, symbol DS90LV011ATMF_NOPB:DS90LV011ATMF_NOPB
- added U14, U16, U17, U18, U19, U21, U22, U9: ~, Resistor_SMD:R_1206_3216Metric, symbol RC1206FR-13330RL:RC1206FR-13330RL
- added U15, U20: AD8052ARMZ-REEL7, part_library:AD8052ARMZ_REEL7, symbol AD8052ARMZ_REEL7:AD8052ARMZ-REEL7
- renumbered C29 to C2, C27 to C3, C32 to C4, C33 to C5, C28 to C6, C26 to C7, R5 to R1, R21 to R10, R9 to R2, R11 to R3, R13 to R4, R15 to R5, R23 to R6, R17 to R7, R1 to R8, R19 to R9, U12 to U1, U11 to U2, U5 to U3, U2 to U8
Connections:
- net GND: now also C24.2, U13.2 (GND), U15.4 (-VS), U20.4 (-VS)
- net VCC_Raw: now also C24.1, U13.1 (VDD), U15.8 (+VS), U20.8 (+VS)
- net 1v8_SPI_NSS: now reaches U8.32 (CSB)
- net 1v8_SPI_CLK: now reaches U8.30 (SCLK)
- net 1v8_SPI_MOSI: now reaches U8.31 (SDIO/PWDN)
- net VCM renamed AD9284_VCM
- net VIN_A_N: no longer names the net of U8.38 (VIN-A)
- net VIN_A_N: now also C42.2, R15.2
- net VIN_A_P: no longer names the net of U8.39 (VIN+A)
- net VIN_A_P: now also C42.1, R14.2
- net VIN_B_N: no longer names the net of U8.47 (VIN-B)
- net VIN_B_N: now also C41.1, R12.2
- net VIN_B_P: no longer names the net of U8.46 (VIN+B)
- net VIN_B_P: now also C41.2, R13.2
- net VREF renamed AD9284_VREF
- net clkn: no longer names the net of U8.33 (CLK-)
- net clkn: now also C28.2
- net clkp: no longer names the net of U8.34 (CLK+)
- net clkp: now also C29.2
- new net: C38.2, U19.2, U20.3 (+IN1)
- new net: C39.2, U20.5 (+IN2), U21.2
- new net: C31.1, U14.2, U16.1
- new net: C35.2, U15.3 (+IN1), U16.2
- new net: C29.1, R11.1, U13.4 (OUT+)
- new net: C28.1, R11.2, U13.3 (OUT-)
- new net: C37.1, U18.2, U19.1
- new net: C37.2, R13.1, U20.1 (OUT1), U20.2 (-IN1)
- new net: C31.2, R15.1, U15.1 (OUT1), U15.2 (-IN1)
- new net: C40.1, U21.1, U22.2
- new net: C40.2, R12.1, U20.6 (-IN2), U20.7 (OUT2)
- new net: C30.1, U17.1, U9.2
- new net: C30.2, R14.1, U15.6 (-IN2), U15.7 (OUT2)
- new net: C36.2, U15.5 (+IN2), U17.2
- new net ADAR_VIN1_N: U9.1
- new net ADAR_VIN1_P: U14.1
- new net ADAR_VIN2_N: U22.1
- new net ADAR_VIN2_P: U18.1
- new net ADAR_VOCM: C35.1, C36.1, C38.1, C39.1
- new net FPGA_CLK: U13.5 (TTLIN)
Other:
- note added: "1n"
- note added: "330 ohm"
- note added: "4.7p"
- note added: "RMCF1206FG100R"
- note added: "[1] Pg. 14"
- note removed: "10uF"
- note removed: "1uF"
- note removed: "3.3v in"
- note removed: "AD9248 BYPASS AND DECOUPLING"
- note removed: "C0603C104K5RACTU"
- note removed: "Clock decoupling"
- note removed: "LDO 1.8V"
- note removed: "Note: MOSI needs to be pulled low post configuration, and CSB/NSS should be held high CLK should be inactive"
- note removed: "POWER SUPPLY"
- note removed: "Pin 41"
- note removed: "Pin 8"
- note removed: "SIGNAL INTEGRITY SHIT"
- note removed: "SPI input and level shifting"
- note removed: "TODO these are kind of just eyeballed with copilot and hints from datasheet. Datasheet shows something more complex but it's probably fine? Running 10MHz max."
- note removed: "VIN decoupling"
- note removed: "[5] Pg. 14"
- note removed: "pin 1, 2"
- note removed: "pin 27"
- note removed: "pin 35 - 37"
- note removed: "pin 42, 40"
- note removed: "pin 43"
- note removed: "pin 44, 45, 48"
- company: (none) -> SD26-11 - Aidan O'Grady
- title: (none) -> ADC Module
- moved on the sheet: C2, C3, C4, C5, C6, C7, R1, R10, R2, R3, R4, R5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

Commit message: Finished and reviewed schematic, one change so far needs to be made: OE pin on level shifters must be externally toggled instead of tied to VCC. The IC requires VDDA/B to be fully ramped before pulling the OE high.
Parts:
- removed C2, C24, C4, C6: C0603C102K5RACTU, part_library:C0603C102K5RACTU, symbol C0603C102K5RACTU:C0603C102K5RACTU
- removed C23, C28, C29, C3, C30, C31, C35, C36, C37, C38, C39, C40, C5, C7: C0603C104K5RACTU, part_library:C0603C104K5RACTU, symbol C0603C104K5RACTU:C0603C104K5RACTU
- removed C41, C42: 06031AR47CAT2A, part_library:06031AR47CAT2A, symbol 06031AR47CAT2A:06031AR47CAT2A
- removed R1, R10, R11, R2, R3, R4, R5, R6, R7, R9: RMCF1206FG100R, part_library:RMCF1206FG100R, symbol RMCF1206FG100R:RMCF1206FG100R
- removed R12, R13, R14, R15: RC1206FR-0733RL, part_library:RC1206FR_0733RL, symbol RC1206FR_0733RL:RC1206FR-0733RL
- removed U1, U2, U3: DS90LV048ATMX/NOPB, part_library:SOIC16, symbol DS9:DS90LV048ATMX_NOPB
- removed U13: DS90LV011ATMF/NOPB, Package_TO_SOT_SMD:SOT-23-5_HandSoldering, symbol DS90LV011ATMF_NOPB:DS90LV011ATMF_NOPB
- removed U14, U16, U17, U18, U19, U21, U22, U9: ~, Resistor_SMD:R_1206_3216Metric, symbol RC1206FR-13330RL:RC1206FR-13330RL
- removed U15, U20: AD8052ARMZ-REEL7, part_library:AD8052ARMZ_REEL7, symbol AD8052ARMZ_REEL7:AD8052ARMZ-REEL7
- added J13, J14, J15, J16, J17, J18, J19, J20, J21, J22: Conn_01x01_Pin, symbol Connector:Conn_01x01_Pin
- renumbered R8 to R1, U8 to U3
Connections:
- net ADC_CLKOUT: now also J15.1 (Pin_1)
- net FPGA_CLK: now also J16.1 (Pin_1)
- net VCC_Analog: no longer U3.1 (AVDD), U3.2 (AVDD), U3.35 (AVDD), U3.36 (AVDD), U3.37 (AVDD), U3.40 (AVDD), U3.42 (AVDD), U3.48 (AVDD)
- net Differential Output Conversion/ADC_DIFFERENTIAL_OUT_7N: now reaches U3.25 (D7-(MSB))
- net Differential Output Conversion/ADC_DIFFERENTIAL_OUT_7P: now reaches U3.26 (D7+(MSB))
- net Differential Output Conversion/ADC_DIFFERENTIAL_OUT_6P: now reaches U3.24 (D6+)
- net Differential Output Conversion/ADC_DIFFERENTIAL_OUT_6N: now reaches U3.23 (D6-)
- net Differential Output Conversion/ADC_DIFFERENTIAL_OUT_5N: now reaches U3.21 (D5-)
- net Differential Output Conversion/ADC_DIFFERENTIAL_OUT_5P: now reaches U3.22 (D5+)
- net Differential Output Conversion/ADC_DIFFERENTIAL_OUT_4P: now reaches U3.20 (D4+)
- net Differential Output Conversion/ADC_DIFFERENTIAL_OUT_4N: now reaches U3.19 (D4-)
- net Differential Output Conversion/ADC_DIFFERENTIAL_OUT_2P: now reaches U3.14 (D2+)
- net Differential Output Conversion/ADC_DIFFERENTIAL_OUT_2N: now reaches U3.13 (D2-)
- net Differential Output Conversion/ADC_DIFFERENTIAL_OUT_1P: now reaches U3.12 (D1+)
- net Differential Output Conversion/ADC_DIFFERENTIAL_OUT_1N: now reaches U3.11 (D1-)
- net Differential Output Conversion/ADC_DIFFERENTIAL_OUT_0P: now reaches U3.10 (D0+(LSB))
- net Differential Output Conversion/ADC_DIFFERENTIAL_OUT_3N: now reaches U3.15 (D3-)
- net Differential Output Conversion/ADC_DIFFERENTIAL_OUT_3P: now reaches U3.16 (D3+)
- net Differential Output Conversion/ADC_DIFFERENTIAL_OUT_DCON: now reaches U3.17 (DCO-)
- net Differential Output Conversion/ADC_DIFFERENTIAL_OUT_DCOP: now reaches U3.18 (DCO+)
- net ADC_CLKN: now reaches U3.33 (CLK-)
- net ADC_CLKN: now also J22.1 (Pin_1)
- net ADC_CLKP: now reaches U3.34 (CLK+)
- net ADC_CLKP: now also J21.1 (Pin_1)
- net ADC_VIN1N: now reaches U3.38 (VIN-A)
- net ADC_VIN1N: now also J20.1 (Pin_1)
- net ADC_VIN1P: now reaches U3.39 (VIN+A)
- net ADC_VIN1P: now also J19.1 (Pin_1)
- net Differential Signal Drivers/ADC_VIN2P: now reaches U3.46 (VIN+B)
- net Differential Signal Drivers/ADC_VIN2N: now reaches U3.47 (VIN-B)
- net Differential Output Conversion/ADC_DIFFERENTIAL_OUT_0N: now reaches U3.9 (D0-(LSB))
- net 1v8_SPI_CLK renamed SPI Level Shifting/1v8_SPI_CLK
- net 1v8_SPI_MOSI renamed SPI Level Shifting/1v8_SPI_MOSI
- net 1v8_SPI_NSS renamed SPI Level Shifting/1v8_SPI_NSS
- net GND renamed gnd
- net VCC_Digital renamed VCC_Digital_1v8
- net VCC_Digital_1v8: now also J13.1 (Pin_1)
- new net ADAR_VIN1N: J18.1 (Pin_1)
- new net ADAR_VIN1P: J17.1 (Pin_1)
- new net VCC_Analog_1v8: J14.1 (Pin_1), U3.1 (AVDD), U3.2 (AVDD), U3.35 (AVDD), U3.36 (AVDD), U3.37 (AVDD), U3.40 (AVDD), U3.42 (AVDD), U3.48 (AVDD)
Other:
- added sheet Differential Output Conversion (Differential_Output_Conversion.kicad_sch)
- added sheet Differential Signal Drivers (Analog_Drivers.kicad_sch)
- added sheet Power Supply and ADC Bypassing (Power_Supply.kicad_sch)
- added sheet SPI Level Shifting (SPI_level_shifting.kicad_sch)
- note added: "ADC High Level Design"
- note added: "ADC Test Points"
- note added: "[1] AD9284 8 bit ADC datasheet: https://www.analog.com/media/en/technical-documentation/data-sheets/ad9284.pdf"
- note removed: "0.001u"
- note removed: "0.1u"
- note removed: "100 ohm"
- note removed: "1n"
- note removed: "33 ohm"
- note removed: "330 ohm"
- note removed: "4.7p"
- note removed: "Mandatory 100 ohm differential impedance prior to reciever input"
- note removed: "RMCF1206FG100R"
- note removed: "[1] Pg. 14"
- note removed: "[4] Pg. 12"
- note removed: "[4] Pg. 13"
- note removed: "[4] Pg. 3"
- moved on the sheet: R1, U3
