File: AD9284/top_level.kicad_sch (KiCad schematic)
At the start: 15 parts, among them J10 Conn_01x01_Pin, J11 Conn_Coaxial, J12 Conn_Coaxial, J13 Conn_Coaxial, J14 Conn_Coaxial, J2 Conn_01x01_Pin, J3 Conn_01x01_Pin, J4 Conn_01x01_Pin, J5 Conn_01x01_Pin, J6 Conn_01x01_Pin, J7 Conn_01x01_Pin, J8 Conn_01x01_Pin, J9 Conn_01x01_Pin, U1 PPPC062LJBN-RC, U2 PPPC062LJBN-RC

Commit message: Schematic and PCB complete. TODO: BOM
Other:
- note removed: "BASYS 3 FPGA to AD9248 connectors (PMOD)"
Changed lines of the file:
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@@
-		)
-	)
-	(text "BASYS 3 FPGA to AD9248 connectors (PMOD)"
-		(exclude_from_sim no)
-		(at 179.578 233.426 0)
-		(effects
-			(font
-				(size 2.54 2.54)
-			)
 		)
 	)
